Commit message: v7.3

File: ros2_ws/src/jetarm_description/urdf/jetarm.urdf.xacro (robot description, xacro)
@@ -11,5 +11,5 @@
   <xacro:property name="j2_upper" value="1.5707963267948966"/>
   <xacro:property name="j3_limit" value="2.0943951023931953"/>
-  <xacro:property name="j4_lower" value="-1.6755160819145563"/>
+  <xacro:property name="j4_lower" value="-2.0943951023931953"/>
   <xacro:property name="j4_upper" value="2.0943951023931953"/>
   <xacro:property name="j5_limit" value="1.0471975511965976"/>

File: ros2_ws/src/jetarm_description/urdf/jetarm_gui.urdf.xacro (robot description, xacro)
@@ -13,5 +13,5 @@
   <xacro:property name="j2_upper" value="1.5707963267948966"/>
   <xacro:property name="j3_limit" value="2.0943951023931953"/>
-  <xacro:property name="j4_lower" value="-1.6755160819145563"/>
+  <xacro:property name="j4_lower" value="-2.0943951023931953"/>
   <xacro:property name="j4_upper" value="2.0943951023931953"/>
   <xacro:property name="j5_limit" value="1.0471975511965976"/>
